File: extension-boards/speaker-board/speaker-board.kicad_sch (KiCad schematic)
At the start: 13 parts, among them J1 Conn_02x04_Odd_Even, U1 LM386

Commit message: Schematic: Silkscreen updated on boards
Parts:
- R1, R2: value 330k -> 300k
Changed lines of the file:
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@@
 			)
 		)
-		(property "Value" "330k"
+		(property "Value" "300k"
 			(at 50.8 50.7999 0)
 			(effects
@@
 			)
 		)
-		(property "Value" "330k"
+		(property "Value" "300k"
 			(at 40.64 50.7999 0)
 			(effects

Commit message: Footprints updated, MPLAB X IDE build configurations updated
Parts:
- C1, C6: footprint Capacitor_THT:CP_Radial_D4.0mm_P2.00mm -> Capacitor_THT:CP_Radial_D5.0mm_P2.00mm
- C5: footprint StockLib:C_100nF_L7.0mm_W2.5mm_P5.00mm -> Capacitor_THT:C_Disc_D3.0mm_W1.6mm_P2.50mm
Changed lines of the file:
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@@
 			)
 		)
-		(property "Footprint" "Capacitor_THT:CP_Radial_D4.0mm_P2.00mm"
+		(property "Footprint" "Capacitor_THT:CP_Radial_D5.0mm_P2.00mm"
 			(at 97.4852 58.42 0)
 			(effects
@@
 			)
 		)
-		(property "Footprint" "StockLib:C_100nF_L7.0mm_W2.5mm_P5.00mm"
+		(property "Footprint" "Capacitor_THT:C_Disc_D3.0mm_W1.6mm_P2.50mm"
 			(at 151.4348 80.01 0)
 			(effects
@@
 			)
 		)
-		(property "Footprint" "Capacitor_THT:CP_Radial_D4.0mm_P2.00mm"
+		(property "Footprint" "Capacitor_THT:CP_Radial_D5.0mm_P2.00mm"
 			(at 178.7652 86.36 0)
 			(effects
